File: iot-mesh.kicad_sch (KiCad schematic)
At the start: 18 parts, among them J1 DS18B20 connector, J2 BME280 connector, J5 Power Connector, U1 XIAO-nRF52840-DIP, U2 WEMOS_D1_mini, U3 L7805

Commit message: Add project specific symbol and footprint
XIAO-nRF52840-DIP is modified so that silkscreen does not go over pads.
Parts:
- removed U1: XIAO-nRF52840-DIP, XIAO_Series_Footprints:XIAO-nRF52840-DIP-mod, symbol Seeed_Studio_XIAO_Series:XIAO-nRF52840-DIP
- added U1: XIAO-nRF52840-DIP, footprints:XIAO-nRF52840-DIP-mk, symbol Seeed_Studio_XIAO_Series_prj:XIAO-nRF52840-DIP
Connections:
- net GND: now also U1.13 (GND)
- net at TP2.1, U2.7 (CS/D8): now also U1.8 (P1.12_D7_RX)
- net at TP1.1, U2.6 (MOSI/D7): now also U1.7 (P1.11_D6_TX)
- net at JP2.1 (A): now also U1.14 (VBUS)
Changed lines of the file:
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@@
+	)
+	(symbol
+		(lib_id "Seeed_Studio_XIAO_Series_prj:XIAO-nRF52840-DIP")
+		(at 119.38 46.99 0)
+		(unit 1)
+		(exclude_from_sim no)
+		(in_bom yes)
+		(on_board yes)
+		(dnp no)
+		(fields_autoplaced yes)
+		(property "Reference" "U1"
+			(at 132.715 43.18 0)
+			(effects
+				(font
+					(size 1.27 1.27)
+				)
+			)
+		)
+		(property "Value" "XIAO-nRF52840-DIP"
+			(at 132.715 45.72 0)
+			(effects
+				(font
+					(size 1.27 1.27)
+				)
+			)
+		)
+		(property "Footprint" "footprints:XIAO-nRF52840-DIP-mk"
+			(at 132.08 77.724 0)
+			(effects
+				(font
+					(size 1.27 1.27)
+				)
+				(hide yes)
+			)
+		)
+		(property "Datasheet" ""
+			(at 115.57 44.45 0)
+			(effects
+				(font
+					(size 1.27 1.27)
+				)
+				(hide yes)
+			)
+		)
+		(property "Description" ""
+			(at 115.57 44.45 0)
+			(effects
+				(font
+					(size 1.27 1.27)
+				)
+				(hide yes)
+			)
+		)
+		(pin "9"
+		)
+		(pin "10"
+		)
+		(pin "8"
+		)
+		(pin "11"
+		)
+		(pin "12"
+		)
+		(pin "1"
+		)
+		(pin "4"
+		)
+		(pin "14"
+		)
+		(pin "13"
+		)
+		(pin "6"
+		)
+		(pin "3"
+		)
+		(pin "5"
+		)
+		(pin "2"
+		)
+		(pin "7"
+		)
+		(instances
+			(project ""
+				(path "/5a2d8fcc-6641-40c3-b318-7df204010f8a"
+					(reference "U1")
+					(unit 1)
+				)
+			)
+		)
 	)
 	(symbol
@@
 					(unit 1)
 				)
-			)
-		)
-	)
-	(symbol
-		(lib_id "Seeed_Studio_XIAO_Series:XIAO-nRF52840-DIP")
-		(at 119.38 46.99 0)
-		(unit 1)
-		(exclude_from_sim no)
-		(in_bom yes)
-		(on_board yes)
-		(dnp no)
-		(fields_autoplaced yes)
-		(property "Reference" "U1"
-			(at 132.715 43.18 0)
-			(effects
-				(font
-					(size 1.27 1.27)
-				)
-			)
-		)
-		(property "Value" "XIAO-nRF52840-DIP"
-			(at 132.715 45.72 0)
-			(effects
-				(font
-					(size 1.27 1.27)
-				)
-			)
-		)
-		(property "Footprint" "XIAO_Series_Footprints:XIAO-nRF52840-DIP-mod"
-			(at 132.08 77.724 0)
-			(effects
-				(font
-					(size 1.27 1.27)
-				)
-				(hide yes)
-			)
-		)
-		(property "Datasheet" ""
-			(at 115.57 44.45 0)
-			(effects
-				(font
-					(size 1.27 1.27)
-				)
-				(hide yes)
-			)
-		)
-		(property "Description" ""
-			(at 115.57 44.45 0)
-			(effects
-				(font
-					(size 1.27 1.27)
-				)
-				(hide yes)
-			)
-		)
-		(pin "13"
-		)
-		(pin "4"
-		)
-		(pin "6"
-		)
-		(pin "7"
-		)
-		(pin "5"
-		)
-		(pin "14"
-		)
-		(pin "12"
-		)
-		(pin "11"
-		)
-		(pin "10"
-		)
-		(pin "9"
-		)
-		(pin "8"
-		)
-		(pin "2"
-		)
-		(pin "1"
-		)
-		(pin "3"
-		)
-		(instances
-			(project ""
-				(path "/5a2d8fcc-6641-40c3-b318-7df204010f8a"
-					(reference "U1")
-					(unit 1)
-				)
