File: iot-mesh.kicad_pcb (KiCad board)
At the start: 2 copper layers, 73 x 39 mm, 18 parts, among them J1 DS18B20 connector, J2 BME280 connector, J5 Power Connector, U1 XIAO-nRF52840-DIP, U2 WEMOS_D1_mini, U3 L7805

Commit message: Component selections and updates for preparing order
Parts:
- R1, R2: footprint Resistor_THT:R_Axial_DIN0207_L6.3mm_D2.5mm_P2.54mm_Vertical -> Resistor_THT:R_Axial_DIN0207_L6.3mm_D2.5mm_P10.16mm_Horizontal
- moved R1 4.58 mm to (137.2, 86.4), turned to -90 degrees
- moved R2 1.80 mm to (133.3, 96.5), turned to 90 degrees
Routing:
- net V_meas_A0: track 53.7 -> 50.6 mm, vias 1 -> 0
Other:
- board text added: "+5V"
